File: 12v-jelly.kicad_pcb (KiCad board)
At the start: 4 copper layers, 46 x 68 mm, 28 parts, among them J1 PWR, J10 8, J3 1, J4 2, J5 3, J6 4, J7 5, J8 6, J9 7, SW2 SW_Push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

Commit message: More tweaks
Parts:
- moved C1 2.87 mm to (86.0, 63.7), turned to 90 degrees
- renumbered H6 to H3, H5 to H4
Connections:
- U2 pad 42: GND -> unconnected-(U2-GND-Pad42)
Routing:
- net GND: track 6.69 -> 14.4 mm, vias 11 -> 9
- net /DATA: track 23.7 -> 26.3 mm
- net +5V: track 24.8 -> 26.1 mm
- net Net-(J1-Pin_2): track 23.7 -> 22.9 mm
- net Net-(J1-Pin_1): track 23.7 -> 22.9 mm

Commit message: More bits
Parts:
- moved FID1 8.00 mm to (80.0, 22.0)
- moved R1 0.10 mm to (91.8, 67.6)
Routing:
- net Net-(J1-Pin_2): track 22.9 -> 26.3 mm
- net Net-(J1-Pin_1): track 22.9 -> 26.3 mm
- net /DATA: track 26.3 -> 24.3 mm, vias 1 -> 0
- net /SW0: track 36.2 -> 37.5 mm
- net /IR: track 21.8 -> 22.3 mm, vias 1 -> 0

Commit message: Tiny tweaks
Parts:
- added kibuzzard-6560DBF2: G***, kibuzzard-6560DBF2, F.Cu at (80.0, 70.0)
Changed lines of the file:
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@@
       (sketchpadsonfab false)
       (subtractmaskfromsilk false)
-      (outputformat 4)
+      (outputformat 1)
       (mirror false)
       (drillshape 0)
@@
       (stroke (width 0.05) (type solid)) (fill none) (layer "F.CrtYd"))
     (pad "" np_thru_hole circle (at 0 0) (size 3.2 3.2) (drill 3.2) (layers "*.Cu" "*.Mask"))
+  )
+  (footprint "kibuzzard-6560DBF2" (layer "F.Cu")
+    (at 80 70)
+    (descr "Generated with KiBuzzard")
+    (tags "kb_params=eyJBbGlnbm1lbnRDaG9pY2UiOiAiQ2VudGVyIiwgIkNhcExlZnRDaG9pY2UiOiAiPCIsICJDYXBSaWdodENob2ljZSI6ICI+IiwgIkZvbnRDb21ib0JveCI6ICJtcGx1cy0xbW4tbWVkaXVtIiwgIkhlaWdodEN0cmwiOiAiMS41IiwgIkxheWVyQ29tYm9Cb3giOiAiRi5TaWxrUyIsICJNdWx0aUxpbmVUZXh0IjogIjEydiBKZWxseSIsICJQYWRkaW5nQm90dG9tQ3RybCI6ICI1IiwgIlBhZGRpbmdMZWZ0Q3RybCI6ICI1IiwgIlBhZGRpbmdSaWdodEN0cmwiOiAiNSIsICJQYWRkaW5nVG9wQ3RybCI6ICI1IiwgIldpZHRoQ3RybCI6ICIifQ==")
+    (attr board_only exclude_from_pos_files exclude_from_bom)
+    (fp_text reference "kibuzzard-6560DBF2" (at 0 -4.687094) (layer "F.SilkS") hide
+        (effects (font (size 0 0)))
+    )
+    (fp_text value "G***" (at 0 4.687094) (layer "F.SilkS") hide
+        (effects (font (size 0 0)))
+    )
+    (fp_poly
+      (pts
+        (xy 0.921544 -0.09525)
+        (xy 1.345406 -0.09525)
+        (xy 1.331119 -0.262235)
+        (xy 1.293019 -0.372666)
+        (xy 1.143 -0.454819)
+        (xy 1.049536 -0.435173)
+        (xy 0.983456 -0.376237)
+        (xy 0.941784 -0.2667)
+        (xy 0.921544 -0.09525)
+      )
+      (stroke (width 0) (type solid)) (fill solid) (layer "F.SilkS"))
+    (fp_poly
+      (pts
+        (xy -5.241131 -1.639094)
+        (xy -5.737225 -1.639094)
+        (xy -6.829954 0)
+        (xy -5.737225 1.639094)
+        (xy -5.241131 1.639094)
+        (xy -4.826794 1.639094)
+        (xy -4.826794 0.619125)
+        (xy -4.826794 -0.869156)
+        (xy -4.831556 -0.871537)
+        (xy -5.241131 -0.642937)
+        (xy -5.241131 -0.8763)
+        (xy -4.824412 -1.119187)
+        (xy -4.560094 -1.119187)
+        (xy -4.560094 0.619125)
+        (xy -4.826794 0.619125)
+        (xy -4.826794 1.639094)
+        (xy -3.2004 1.639094)
+        (xy -3.2004 0.619125)
+        (xy -4.05765 0.619125)
+        (xy -4.05765 0.411956)
+        (xy -3.904764 0.234237)
+        (xy -3.775399 0.064391)
+        (xy -3.669555 -0.097583)
+        (xy -3.587232 -0.251684)
+        (xy -3.528429 -0.397912)
+        (xy -3.493148 -0.536267)
+        (xy -3.481387 -0.66675)
+        (xy -3.494187 -0.788194)
+        (xy -3.532584 -0.871537)
+        (xy -3.688556 -0.935831)
+        (xy -3.800475 -0.920221)
+        (xy -3.923506 -0.87339)
+        (xy -4.05765 -0.795337)
+        (xy -4.05765 -1.019175)
+        (xy -3.925887 -1.087967)
+        (xy -3.7846 -1.129242)
+        (xy -3.633787 -1.143)
+        (xy -3.45311 -1.113532)
+        (xy -3.320653 -1.025128)
+        (xy -3.239393 -0.879574)
+        (xy -3.212306 -0.678656)
+        (xy -3.227255 -0.527844)
+        (xy -3.272102 -0.367506)
+        (xy -3.346847 -0.197644)
+        (xy -3.424461 -0.061615)
+        (xy -3.522762 0.084534)
+        (xy -3.64175 0.240804)
+        (xy -3.781425 0.407194)
+        (xy -3.781425 0.411956)
+        (xy -3.2004 0.411956)
+        (xy -3.2004 0.619125)
+        (xy -3.2004 1.639094)
+        (xy -2.271712 1.639094)
+        (xy -2.271712 0.619125)
+        (xy -2.605087 0.619125)
+        (xy -2.938462 -0.619125)
+        (xy -2.667 -0.619125)
+        (xy -2.436019 0.428625)
+        (xy -2.431256 0.428625)
+        (xy -2.200275 -0.619125)
+        (xy -1.938337 -0.619125)
+        (xy -2.271712 0.619125)
+        (xy -2.271712 1.639094)
+        (xy -0.17145 1.639094)
+        (xy -0.17145 0.642938)
+        (xy -0.363141 0.623888)
+        (xy -0.5334 0.566738)
+        (xy -0.5334 0.345281)
+        (xy -0.360759 0.409575)
+        (xy -0.195262 0.435769)
+        (xy -0.086916 0.421481)
+        (xy -0.014287 0.378619)
+        (xy 0.026789 0.299442)
+        (xy 0.040481 0.176213)
+        (xy 0.040481 -0.912019)
+        (xy -0.3429 -0.912019)
+        (xy -0.3429 -1.119187)
+        (xy 0.311944 -1.119187)
+        (xy 0.311944 0.185737)
+        (xy 0.30017 0.340916)
+        (xy 0.264848 0.460375)
+        (xy 0.205978 0.544116)
+        (xy 0.116946 0.599017)
+        (xy -0.008864 0.631957)
+        (xy -0.17145 0.642938)
+        (xy -0.17145 1.639094)
+        (xy 1.197769 1.639094)
+        (xy 1.197769 0.642938)
+        (xy 1.03042 0.625078)
+        (xy 0.893498 0.5715)
+        (xy 0.787003 0.482203)
+        (xy 0.710935 0.357188)
+        (xy 0.665295 0.196453)
+        (xy 0.650081 0)
+        (xy 0.663972 -0.196453)
+        (xy 0.705644 -0.357187)
+        (xy 0.775097 -0.482203)
+        (xy 0.872331 -0.5715)
+        (xy 0.997347 -0.625078)
+        (xy 1.150144 -0.642937)
+        (xy 1.289579 -0.626136)
+        (xy 1.403085 -0.575733)
+        (xy 1.490663 -0.491728)
+        (xy 1.55284 -0.370417)
+        (xy 1.590146 -0.208095)
+        (xy 1.602581 -0.004762)
+        (xy 1.597819 0.090488)
+        (xy 0.921544 0.090488)
+        (xy 0.949226 0.257473)
+        (xy 1.008459 0.367903)
+        (xy 1.10103 0.429518)
+        (xy 1.228725 0.450056)
+        (xy 1.375172 0.433983)
+        (xy 1.538288 0.385763)
+        (xy 1.538288 0.583406)
+        (xy 1.363861 0.628055)
+        (xy 1.197769 0.642938)
+        (xy 1.197769 1.639094)
+        (xy 2.764631 1.639094)
+        (xy 2.764631 0.619125)
+        (xy 2.178844 0.619125)
+        (xy 2.178844 -0.926306)
+        (xy 1.859756 -0.926306)
+        (xy 1.859756 -1.119187)
+        (xy 2.445544 -1.119187)
+        (xy 2.445544 0.426244)
+        (xy 2.764631 0.426244)
+        (xy 2.764631 0.619125)
+        (xy 2.764631 1.639094)
+        (xy 3.955256 1.639094)
+        (xy 3.955256 0.619125)
+        (xy 3.369469 0.619125)
+        (xy 3.369469 -0.926306)
+        (xy 3.050381 -0.926306)
+        (xy 3.050381 -1.119187)
+        (xy 3.636169 -1.119187)
+        (xy 3.636169 0.426244)
+        (xy 3.955256 0.426244)
+        (xy 3.955256 0.619125)
+        (xy 3.955256 1.639094)
+        (xy 4.672013 1.639094)
+        (xy 4.672013 1.143)
+        (xy 4.410075 1.143)
+        (xy 4.605338 0.595313)
+        (xy 4.193381 -0.619125)
+        (xy 4.452938 -0.619125)
+        (xy 4.717256 0.28575)
+        (xy 4.722019 0.28575)
+        (xy 4.969669 -0.619125)
+        (xy 5.241131 -0.619125)
+        (xy 4.672013 1.143)
+        (xy 4.672013 1.639094)
+        (xy 5.241131 1.639094)
+        (xy 5.737225 1.639094)
+        (xy 6.829954 0)
+        (xy 5.737225 -1.639094)
+        (xy 5.241131 -1.639094)
+        (xy -5.241131 -1.639094)
+      )
+      (stroke (width 0) (type solid)) (fill solid) (layer "F.SilkS"))
   )
   (footprint "Fiducial:Fiducial_1mm_Mask2mm" (layer "F.Cu")
@@
     (polygon
       (pts
-        (xy 77.5 55.35)
-        (xy 82.5 55.35)
+        (xy 77.5 52.85)
+        (xy 82.5 52.85)
         (xy 82.5 77.575)
         (xy 77.5 77.575)
