File: 12v-jelly.kicad_sch (KiCad schematic)
At the start: 30 parts, among them J1 PWR, J10 8, J3 1, J4 2, J5 3, J6 4, J7 5, J8 6, J9 7, SW2 SW_Push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

Commit message: Double Sided layout and further tweaks
Parts:
- removed H3, H4: MountingHole, MountingHole:MountingHole_3.2mm_M3, symbol Mechanical:MountingHole
Other:
- moved on the sheet: FID1, FID2, FID3
Changed lines of the file:
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@@
     (effects (font (size 1.27 1.27)) (justify left bottom))
   )
-  (symbol (lib_id "Mechanical:MountingHole") (at 17.78 43.18 0) (unit 1)
-    (in_bom yes) (on_board yes) (dnp no) (fields_autoplaced)
-    (property "Reference" "H4" (at 20.32 42.3453 0)
-      (effects (font (size 1.27 1.27)) (justify left))
-    )
-    (property "Value" "MountingHole" (at 20.32 44.8822 0)
-      (effects (font (size 1.27 1.27)) (justify left))
-    )
-    (property "Footprint" "MountingHole:MountingHole_3.2mm_M3" (at 17.78 43.18 0)
+  (symbol (lib_id "power:+5V") (at 259.08 26.67 0) (unit 1)
+    (in_bom yes) (on_board yes) (dnp no) (fields_autoplaced)
+    (property "Reference" "#PWR03" (at 259.08 30.48 0)
+      (effects (font (size 1.27 1.27)) hide)
+    )
+    (property "Value" "+5V" (at 259.08 23.0942 0)
+      (effects (font (size 1.27 1.27)))
+    )
+    (property "Footprint" "" (at 259.08 26.67 0)
+      (effects (font (size 1.27 1.27)) hide)
+    )
+    (property "Datasheet" "" (at 259.08 26.67 0)
+      (effects (font (size 1.27 1.27)) hide)
+    )
+    (pin "1")
+    (instances
+      (project "porta-jelly"
+        (path "/10477f3c-6568-4c00-b643-b8ffee73b374"
+          (reference "#PWR03") (unit 1)
+        )
+      )
+      (project "12v-jelly"
+        (path "/a6bbc090-914d-4858-aeca-5d2d4d192127"
+          (reference "#PWR03") (unit 1)
+        )
+      )
+      (project ""
+        (path "/d350497a-baf4-4270-a560-45c7bc5aa03e"
+          (reference "#PWR03") (unit 1)
+        )
+      )
+    )
+  )
+  (symbol (lib_id "Mechanical:Fiducial") (at 17.78 43.18 0) (unit 1)
+    (in_bom yes) (on_board yes) (dnp no) (fields_autoplaced)
+    (property "Reference" "FID2" (at 19.939 42.5363 0)
+      (effects (font (size 1.27 1.27)) (justify left))
+    )
+    (property "Value" "Fiducial" (at 19.939 44.4573 0)
+      (effects (font (size 1.27 1.27)) (justify left))
+    )
+    (property "Footprint" "Fiducial:Fiducial_1mm_Mask2mm" (at 17.78 43.18 0)
       (effects (font (size 1.27 1.27)) hide)
     )
     (property "Datasheet" "~" (at 17.78 43.18 0)
-      (effects (font (size 1.27 1.27)) hide)
-    )
-    (instances
-      (project "porta-jelly"
-        (path "/10477f3c-6568-4c00-b643-b8ffee73b374"
-          (reference "H4") (unit 1)
-        )
-      )
-      (project "12v-jelly"
-        (path "/a6bbc090-914d-4858-aeca-5d2d4d192127"
-          (reference "H6") (unit 1)
-        )
-      )
-      (project ""
-        (path "/d350497a-baf4-4270-a560-45c7bc5aa03e"
-          (reference "H4") (unit 1)
-        )
-      )
-    )
-  )
-  (symbol (lib_id "power:+5V") (at 259.08 26.67 0) (unit 1)
-    (in_bom yes) (on_board yes) (dnp no) (fields_autoplaced)
-    (property "Reference" "#PWR03" (at 259.08 30.48 0)
-      (effects (font (size 1.27 1.27)) hide)
-    )
-    (property "Value" "+5V" (at 259.08 23.0942 0)
-      (effects (font (size 1.27 1.27)))
-    )
-    (property "Footprint" "" (at 259.08 26.67 0)
-      (effects (font (size 1.27 1.27)) hide)
-    )
-    (property "Datasheet" "" (at 259.08 26.67 0)
-      (effects (font (size 1.27 1.27)) hide)
-    )
-    (pin "1")
-    (instances
-      (project "porta-jelly"
-        (path "/10477f3c-6568-4c00-b643-b8ffee73b374"
-          (reference "#PWR03") (unit 1)
-        )
-      )
-      (project "12v-jelly"
-        (path "/a6bbc090-914d-4858-aeca-5d2d4d192127"
-          (reference "#PWR03") (unit 1)
-        )
-      )
-      (project ""
-        (path "/d350497a-baf4-4270-a560-45c7bc5aa03e"
-          (reference "#PWR03") (unit 1)
-        )
-      )
-    )
-  )
-  (symbol (lib_id "Mechanical:Fiducial") (at 17.78 53.34 0) (unit 1)
-    (in_bom yes) (on_board yes) (dnp no) (fields_autoplaced)
-    (property "Reference" "FID2" (at 19.939 52.6963 0)
-      (effects (font (size 1.27 1.27)) (justify left))
-    )
-    (property "Value" "Fiducial" (at 19.939 54.6173 0)
-      (effects (font (size 1.27 1.27)) (justify left))
-    )
-    (property "Footprint" "Fiducial:Fiducial_1mm_Mask2mm" (at 17.78 53.34 0)
-      (effects (font (size 1.27 1.27)) hide)
-    )
-    (property "Datasheet" "~" (at 17.78 53.34 0)
       (effects (font (size 1.27 1.27)) hide)
     )
@@
     )
   )
-  (symbol (lib_id "Mechanical:Fiducial") (at 17.78 58.42 0) (unit 1)
-    (in_bom yes) (on_board yes) (dnp no) (fields_autoplaced)
-    (property "Reference" "FID3" (at 19.939 57.7763 0)
-      (effects (font (size 1.27 1.27)) (justify left))
-    )
-    (property "Value" "Fiducial" (at 19.939 59.6973 0)
-      (effects (font (size 1.27 1.27)) (justify left))
-    )
-    (property "Footprint" "Fiducial:Fiducial_1mm_Mask2mm" (at 17.78 58.42 0)
-      (effects (font (size 1.27 1.27)) hide)
-    )
-    (property "Datasheet" "~" (at 17.78 58.42 0)
+  (symbol (lib_id "Mechanical:Fiducial") (at 17.78 48.26 0) (unit 1)
+    (in_bom yes) (on_board yes) (dnp no) (fields_autoplaced)
+    (property "Reference" "FID3" (at 19.939 47.6163 0)
+      (effects (font (size 1.27 1.27)) (justify left))
+    )
+    (property "Value" "Fiducial" (at 19.939 49.5373 0)
+      (effects (font (size 1.27 1.27)) (justify left))
+    )
+    (property "Footprint" "Fiducial:Fiducial_1mm_Mask2mm" (at 17.78 48.26 0)
+      (effects (font (size 1.27 1.27)) hide)
+    )
+    (property "Datasheet" "~" (at 17.78 48.26 0)
       (effects (font (size 1.27 1.27)) hide)
     )
@@
         (path "/a6bbc090-914d-4858-aeca-5d2d4d192127"
           (reference "FID3") (unit 1)
-        )
-      )
-    )
-  )
-  (symbol (lib_id "Mechanical:MountingHole") (at 17.78 38.1 0) (unit 1)
-    (in_bom yes) (on_board yes) (dnp no) (fields_autoplaced)
-    (property "Reference" "H3" (at 20.32 37.2653 0)
-      (effects (font (size 1.27 1.27)) (justify left))
-    )
-    (property "Value" "MountingHole" (at 20.32 39.8022 0)
-      (effects (font (size 1.27 1.27)) (justify left))
-    )
-    (property "Footprint" "MountingHole:MountingHole_3.2mm_M3" (at 17.78 38.1 0)
-      (effects (font (size 1.27 1.27)) hide)
-    )
-    (property "Datasheet" "~" (at 17.78 38.1 0)
-      (effects (font (size 1.27 1.27)) hide)
-    )
-    (instances
-      (project "porta-jelly"
-        (path "/10477f3c-6568-4c00-b643-b8ffee73b374"
-          (reference "H3") (unit 1)
-        )
-      )
-      (project "12v-jelly"
-        (path "/a6bbc090-914d-4858-aeca-5d2d4d192127"
-          (reference "H5") (unit 1)
-        )
-      )
-      (project ""
-        (path "/d350497a-baf4-4270-a560-45c7bc5aa03e"
-          (reference "H3") (unit 1)
         )
       )
@@
     )
   )
-  (symbol (lib_id "Mechanical:Fiducial") (at 17.78 48.26 0) (unit 1)
-    (in_bom yes) (on_board yes) (dnp no) (fields_autoplaced)
-    (property "Reference" "FID1" (at 19.939 47.6163 0)
-      (effects (font (size 1.27 1.27)) (justify left))
-    )
-    (property "Value" "Fiducial" (at 19.939 49.5373 0)
-      (effects (font (size 1.27 1.27)) (justify left))
-    )
-    (property "Footprint" "Fiducial:Fiducial_1mm_Mask2mm" (at 17.78 48.26 0)
-      (effects (font (size 1.27 1.27)) hide)
-    )
-    (property "Datasheet" "~" (at 17.78 48.26 0)
-      (effects (font (size 1.27 1.27)) hide)
-    )
+  (symbol (lib_id "Mechanical:Fiducial") (at 17.78 38.1 0) (unit 1)
+    (in_bom yes) (on_board yes) (dnp no) (fields_autoplaced)
+    (property "Reference" "FID1" (at 19.939 37.4563 0)
+      (effects (font (size 1.27 1.27)) (justify left))
+    )
+    (property "Value" "Fiducial" (at 19.939 39.3773 0)
+      (effects (font (size 1.27 1.27)) (justify left))
+    )
+    (property "Footprint" "Fiducial:Fiducial_1mm_Mask2mm" (at 17.78 38.1 0)
+      (effects (font (size 1.27 1.27)) hide)
+    )
+    (property "Datasheet" "~" (at 17.78 38.1 0)
+      (effects (font (size 1.27 1.27)) hide)
+    )

Commit message: More tweaks
Parts:
- U2: footprint MCU_RaspberryPi_and_Boards:RPi_Pico_SMD_TH -> MCU_RaspberryPi_and_Boards:RPi_Pico_SMD
Connections:
- net GND: no longer U2.42 (GND)
- no-connect marks 29 -> 30
Changed lines of the file:
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@@
   (no_connect (at 167.64 40.64))
   (no_connect (at 167.64 43.18))
+  (no_connect (at 185.42 81.28))
   (no_connect (at 104.14 66.04))
   (wire (pts (xy 227.33 43.18) (xy 236.22 43.18))
@@
   )
   (wire (pts (xy 262.89 104.14) (xy 248.92 104.14))
-    (stroke (width 0) (type default))
-  )
-  (wire (pts (xy 185.42 82.55) (xy 185.42 81.28))
     (stroke (width 0) (type default))
   )
@@
       (effects (font (size 1.27 1.27)))
     )
-    (property "Footprint" "MCU_RaspberryPi_and_Boards:RPi_Pico_SMD_TH" (at 185.42 52.07 90)
-      (effects (font (size 1.27 1.27)) hide)
-    )
+    (property "Footprint" "MCU_RaspberryPi_and_Boards:RPi_Pico_SMD" (at 185.42 52.07 90)
+      (effects (font (size 1.27 1.27)) hide)
+    )

Commit message: MOSFET
Parts:
- added Q1: Q_NMOS_GDS, Package_TO_SOT_SMD:TO-252-3_TabPin2, symbol Device:Q_NMOS_GDS
- added R1: 10k, Resistor_SMD:R_0603_1608Metric, symbol Device:R_Small
Connections:
- net +5V: now also Q1.2 (D); no longer C1.1, J10.3 (Pin_3), J3.3 (Pin_3), J4.3 (Pin_3), J5.3 (Pin_3), J6.3 (Pin_3), J7.3 (Pin_3), J8.3 (Pin_3), J9.3 (Pin_3), U1.10 (~{SRCLR}), U1.16 (VCC)
- net GND: now also R1.2
- net LED_EN: now reaches U2.2 (GPIO1)
- net LED_EN: now also Q1.1 (G), R1.1
- new net LED_PWR: C1.1, J10.3 (Pin_3), J3.3 (Pin_3), J4.3 (Pin_3), J5.3 (Pin_3), J6.3 (Pin_3), J7.3 (Pin_3), J8.3 (Pin_3), J9.3 (Pin_3), Q1.3 (S), U1.10 (~{SRCLR}), U1.16 (VCC)
- no-connect marks 30 -> 29
Other:
- moved on the sheet: J1, U3

Commit message: PMOS not NMOS
Parts:
- removed Q1: Q_NMOS_GDS, Package_TO_SOT_SMD:TO-252-3_TabPin2, symbol Device:Q_NMOS_GDS
- added Q1: DMP2022LSS-13, Package_SO:SO-8_3.9x4.9mm_P1.27mm, symbol 12v-jelly:DMP2022LSS-13
Connections:
- net +5V: now also R1.1, Q1.1 (S), Q1.2 (S), Q1.3 (S)
- net GND: no longer R1.2
- net LED_EN: now also R1.2, Q1.4 (G); no longer R1.1
- net LED_PWR: now also Q1.5 (D), Q1.6 (D), Q1.7 (D), Q1.8 (D)
Other:
- moved on the sheet: R1
Changed lines of the file:
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@@
   (junction (at 185.42 82.55) (diameter 0) (color 0 0 0 0)
   )
+  (junction (at 99.06 66.04) (diameter 0) (color 0 0 0 0)
+  )
   (junction (at 259.08 66.04) (diameter 0) (color 0 0 0 0)
   )
   (junction (at 261.62 40.64) (diameter 0) (color 0 0 0 0)
   )
+  (junction (at 259.08 35.56) (diameter 0) (color 0 0 0 0)
+  )
+  (junction (at 72.39 25.4) (diameter 0) (color 0 0 0 0)
+  )
+  (junction (at 259.08 45.72) (diameter 0) (color 0 0 0 0)
+  )
   (junction (at 106.68 73.66) (diameter 0) (color 0 0 0 0)
-  )
-  (junction (at 259.08 35.56) (diameter 0) (color 0 0 0 0)
-  )
-  (junction (at 72.39 25.4) (diameter 0) (color 0 0 0 0)
-  )
-  (junction (at 259.08 45.72) (diameter 0) (color 0 0 0 0)
   )
   (junction (at 259.08 55.88) (diameter 0) (color 0 0 0 0)
@@
     (stroke (width 0) (type default))
   )
+  (wire (pts (xy 106.68 73.66) (xy 99.06 73.66))
+    (stroke (width 0) (type default))
+  )
   (wire (pts (xy 243.84 25.4) (xy 243.84 26.67))
     (stroke (width 0) (type default))
@@
     (stroke (width 0) (type default))
   )
-  (wire (pts (xy 92.71 66.04) (xy 101.6 66.04))
+  (wire (pts (xy 92.71 66.04) (xy 99.06 66.04))
     (stroke (width 0) (type default))
   )
@@
     (stroke (width 0) (type default))
   )
+  (wire (pts (xy 99.06 66.04) (xy 99.06 67.31))
+    (stroke (width 0) (type default))
+  )
   (wire (pts (xy 261.62 40.64) (xy 262.89 40.64))
     (stroke (width 0) (type default))
@@
     (stroke (width 0) (type default))
   )
+  (wire (pts (xy 99.06 73.66) (xy 99.06 72.39))
+    (stroke (width 0) (type default))
+  )
   (wire (pts (xy 210.82 71.12) (xy 203.2 71.12))
     (stroke (width 0) (type default))
@@
   )
   (wire (pts (xy 214.63 38.1) (xy 214.63 36.83))
+    (stroke (width 0) (type default))
+  )
+  (wire (pts (xy 99.06 66.04) (xy 101.6 66.04))
     (stroke (width 0) (type default))
   )
@@
     (property "Intersheetrefs" "${INTERSHEET_REFS}" (at 243.84 14.0881 90)
       (effects (font (size 1.27 1.27)) (justify left) hide)
+    )
+  )
+  (symbol (lib_id "12v-jelly:DMP2022LSS-13") (at 106.68 68.58 270) (mirror x) (unit 1)
+    (in_bom yes) (on_board yes) (dnp no) (fields_autoplaced)
+    (property "Reference" "Q1" (at 106.68 61.1251 90)
+      (effects (font (size 1.27 1.27)))
+    )
+    (property "Value" "DMP2022LSS-13" (at 106.68 63.0461 90)
+      (effects (font (size 1.27 1.27)))
+    )
+    (property "Footprint" "Package_SO:SO-8_3.9x4.9mm_P1.27mm" (at 109.22 63.5 0)
+      (effects (font (size 1.27 1.27)) hide)
+    )
+    (property "Datasheet" "~" (at 106.68 68.58 0)
+      (effects (font (size 1.27 1.27)) hide)
+    )
+    (pin "1")
+    (pin "2")
+    (pin "3")
+    (pin "4")
+    (pin "5")
+    (pin "6")
+    (pin "7")
+    (pin "8")
+    (instances
+      (project "12v-jelly"
+        (path "/a6bbc090-914d-4858-aeca-5d2d4d192127"
+          (reference "Q1") (unit 1)
+        )
+      )
     )
   )
@@
         (path "/a6bbc090-914d-4858-aeca-5d2d4d192127"
           (reference "FID3") (unit 1)
-        )
-      )
-    )
-  )
-  (symbol (lib_id "Device:Q_NMOS_GDS") (at 106.68 68.58 90) (unit 1)
-    (in_bom yes) (on_board yes) (dnp no) (fields_autoplaced)
-    (property "Reference" "Q1" (at 106.68 61.1251 90)
-      (effects (font (size 1.27 1.27)))
-    )
-    (property "Value" "Q_NMOS_GDS" (at 106.68 63.0461 90)
-      (effects (font (size 1.27 1.27)))
-    )
-    (property "Footprint" "Package_TO_SOT_SMD:TO-252-3_TabPin2" (at 104.14 63.5 0)
-      (effects (font (size 1.27 1.27)) hide)
-    )
-    (property "Datasheet" "~" (at 106.68 68.58 0)
-      (effects (font (size 1.27 1.27)) hide)
-    )
-    (pin "1")
-    (pin "2")
-    (pin "3")
-    (instances
-      (project "12v-jelly"
-        (path "/a6bbc090-914d-4858-aeca-5d2d4d192127"
-          (reference "Q1") (unit 1)
         )
       )
@@
     )
   )
-  (symbol (lib_id "power:GND") (at 106.68 78.74 0) (unit 1)
-    (in_bom yes) (on_board yes) (dnp no) (fields_autoplaced)
-    (property "Reference" "#PWR08" (at 106.68 85.09 0)
-      (effects (font (size 1.27 1.27)) hide)
-    )
-    (property "Value" "GND" (at 106.68 83.1834 0)
-      (effects (font (size 1.27 1.27)))
-    )
-    (property "Footprint" "" (at 106.68 78.74 0)
-      (effects (font (size 1.27 1.27)) hide)
-    )
-    (property "Datasheet" "" (at 106.68 78.74 0)
-      (effects (font (size 1.27 1.27)) hide)
-    )
-    (pin "1")
-    (instances
-      (project "porta-jelly"
-        (path "/10477f3c-6568-4c00-b643-b8ffee73b374"
-          (reference "#PWR08") (unit 1)
-        )
-      )
-      (project "12v-jelly"
-        (path "/a6bbc090-914d-4858-aeca-5d2d4d192127"
-          (reference "#PWR03") (unit 1)
-        )
-      )
-      (project ""
-        (path "/d350497a-baf4-4270-a560-45c7bc5aa03e"
-          (reference "#PWR0102") (unit 1)
-        )
-      )
-    )
-  )
   (symbol (lib_id "power:GND") (at 130.81 40.64 0) (unit 1)
     (in_bom yes) (on_board yes) (dnp no) (fields_autoplaced)
@@
     )
   )
-  (symbol (lib_id "Device:R_Small") (at 106.68 76.2 0) (unit 1)
-    (in_bom yes) (on_board yes) (dnp no) (fields_autoplaced)
-    (property "Reference" "R1" (at 108.1786 75.5563 0)
-      (effects (font (size 1.27 1.27)) (justify left))
-    )
-    (property "Value" "10k" (at 108.1786 77.4773 0)
-      (effects (font (size 1.27 1.27)) (justify left))
-    )
-    (property "Footprint" "Resistor_SMD:R_0603_1608Metric" (at 106.68 76.2 0)
-      (effects (font (size 1.27 1.27)) hide)
-    )
-    (property "Datasheet" "~" (at 106.68 76.2 0)
-      (effects (font (size 1.27 1.27)) hide)
-    )
+  (symbol (lib_id "Device:R_Small") (at 99.06 69.85 0) (unit 1)
+    (in_bom yes) (on_board yes) (dnp no) (fields_autoplaced)
+    (property "Reference" "R1" (at 100.5586 69.2063 0)
+      (effects (font (size 1.27 1.27)) (justify left))
+    )
+    (property "Value" "10k" (at 100.5586 71.1273 0)
+      (effects (font (size 1.27 1.27)) (justify left))
+    )
+    (property "Footprint" "Resistor_SMD:R_0603_1608Metric" (at 99.06 69.85 0)
+      (effects (font (size 1.27 1.27)) hide)
+    )
+    (property "Datasheet" "~" (at 99.06 69.85 0)
+      (effects (font (size 1.27 1.27)) hide)
+    )

Commit message: Driver NMOS
Parts:
- added Q2: 2N7002, Package_TO_SOT_SMD:SOT-23, symbol Transistor_FET:2N7002
- added R1: 10k, Resistor_SMD:R_0603_1608Metric, symbol Device:R_Small
Connections:
- net GND: now also Q2.2 (S), R1.2
- net LED_EN: now also Q2.1 (G), R1.1; no longer Q1.4 (G), R1.2
- new net: Q1.4 (G), Q2.3 (D), R1.2
Changed lines of the file:
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@@
   (junction (at 259.08 45.72) (diameter 0) (color 0 0 0 0)
   )
+  (junction (at 259.08 55.88) (diameter 0) (color 0 0 0 0)
+  )
+  (junction (at 261.62 71.12) (diameter 0) (color 0 0 0 0)
+  )
+  (junction (at 92.71 66.04) (diameter 0) (color 0 0 0 0)
+  )
+  (junction (at 160.02 71.12) (diameter 0) (color 0 0 0 0)
+  )
+  (junction (at 259.08 96.52) (diameter 0) (color 0 0 0 0)
+  )
+  (junction (at 259.08 86.36) (diameter 0) (color 0 0 0 0)
+  )
   (junction (at 106.68 73.66) (diameter 0) (color 0 0 0 0)
-  )
-  (junction (at 259.08 55.88) (diameter 0) (color 0 0 0 0)
-  )
-  (junction (at 261.62 71.12) (diameter 0) (color 0 0 0 0)
-  )
-  (junction (at 92.71 66.04) (diameter 0) (color 0 0 0 0)
-  )
-  (junction (at 160.02 71.12) (diameter 0) (color 0 0 0 0)
-  )
-  (junction (at 259.08 96.52) (diameter 0) (color 0 0 0 0)
-  )
-  (junction (at 259.08 86.36) (diameter 0) (color 0 0 0 0)
   )
   (junction (at 236.22 88.9) (diameter 0) (color 0 0 0 0)
@@
     (stroke (width 0) (type default))
   )
-  (wire (pts (xy 106.68 73.66) (xy 110.49 73.66))
-    (stroke (width 0) (type default))
-  )
   (wire (pts (xy 259.08 55.88) (xy 262.89 55.88))
     (stroke (width 0) (type default))
@@
     (effects (font (size 1.27 1.27)) (justify right bottom))
   )
+  (label "LED_EN" (at 114.3 78.74 0) (fields_autoplaced)
+    (effects (font (size 1.27 1.27)) (justify left bottom))
+  )
   (label "CLOCK" (at 223.52 64.77 180) (fields_autoplaced)
     (effects (font (size 1.27 1.27)) (justify right bottom))
@@
   (label "LED_EN" (at 167.64 30.48 180) (fields_autoplaced)
     (effects (font (size 1.27 1.27)) (justify right bottom))
-  )
-  (label "LED_EN" (at 110.49 73.66 0) (fields_autoplaced)
-    (effects (font (size 1.27 1.27)) (justify left bottom))
   )
   (label "SW0" (at 80.01 25.4 0) (fields_autoplaced)
@@
         (path "/d350497a-baf4-4270-a560-45c7bc5aa03e"
           (reference "J9") (unit 1)
+        )
+      )
+    )
+  )
+  (symbol (lib_id "Transistor_FET:2N7002") (at 109.22 78.74 0) (mirror y) (unit 1)
+    (in_bom yes) (on_board yes) (dnp no) (fields_autoplaced)
+    (property "Reference" "Q2" (at 104.013 78.0963 0)
+      (effects (font (size 1.27 1.27)) (justify left))
+    )
+    (property "Value" "2N7002" (at 104.013 80.0173 0)
+      (effects (font (size 1.27 1.27)) (justify left))
+    )
+    (property "Footprint" "Package_TO_SOT_SMD:SOT-23" (at 104.14 80.645 0)
+      (effects (font (size 1.27 1.27) italic) (justify left) hide)
+    )
+    (property "Datasheet" "https://www.onsemi.com/pub/Collateral/NDS7002A-D.PDF" (at 109.22 78.74 0)
+      (effects (font (size 1.27 1.27)) (justify left) hide)
+    )
+    (pin "1")
+    (pin "2")
+    (pin "3")
+    (instances
+      (project "12v-jelly"
+        (path "/a6bbc090-914d-4858-aeca-5d2d4d192127"
+          (reference "Q2") (unit 1)
         )
       )
@@
     )
   )
+  (symbol (lib_id "power:GND") (at 114.3 83.82 0) (unit 1)
+    (in_bom yes) (on_board yes) (dnp no) (fields_autoplaced)
+    (property "Reference" "#PWR09" (at 114.3 90.17 0)
+      (effects (font (size 1.27 1.27)) hide)
+    )
+    (property "Value" "GND" (at 114.3 88.2634 0)
+      (effects (font (size 1.27 1.27)))
+    )
+    (property "Footprint" "" (at 114.3 83.82 0)
+      (effects (font (size 1.27 1.27)) hide)
+    )
+    (property "Datasheet" "" (at 114.3 83.82 0)
+      (effects (font (size 1.27 1.27)) hide)
+    )
+    (pin "1")
+    (instances
+      (project "porta-jelly"
+        (path "/10477f3c-6568-4c00-b643-b8ffee73b374"
+          (reference "#PWR09") (unit 1)
+        )
+      )
+      (project "12v-jelly"
+        (path "/a6bbc090-914d-4858-aeca-5d2d4d192127"
+          (reference "#PWR06") (unit 1)
+        )
+      )
+      (project ""
+        (path "/d350497a-baf4-4270-a560-45c7bc5aa03e"
+          (reference "#PWR09") (unit 1)
+        )
+      )
+    )
+  )
+  (symbol (lib_id "Device:R_Small") (at 114.3 81.28 0) (unit 1)
+    (in_bom yes) (on_board yes) (dnp no) (fields_autoplaced)
+    (property "Reference" "R1" (at 115.7986 80.6363 0)
+      (effects (font (size 1.27 1.27)) (justify left))
+    )
+    (property "Value" "10k" (at 115.7986 82.5573 0)
+      (effects (font (size 1.27 1.27)) (justify left))
+    )
+    (property "Footprint" "Resistor_SMD:R_0603_1608Metric" (at 114.3 81.28 0)
+      (effects (font (size 1.27 1.27)) hide)
+    )
+    (property "Datasheet" "~" (at 114.3 81.28 0)
+      (effects (font (size 1.27 1.27)) hide)
+    )
+    (pin "1")
+    (pin "2")
+    (instances
+      (project "porta-jelly"
+        (path "/10477f3c-6568-4c00-b643-b8ffee73b374"
+          (reference "R1") (unit 1)
+        )
+      )
+      (project "12v-jelly"
+        (path "/a6bbc090-914d-4858-aeca-5d2d4d192127"
+          (reference "R5") (unit 1)
+        )
+      )
+    )
+  )
   (symbol (lib_id "power:GND") (at 93.98 27.94 0) (unit 1)
     (in_bom yes) (on_board yes) (dnp no) (fields_autoplaced)
@@
         )
       )
+    )
+  )
+  (symbol (lib_id "power:GND") (at 106.68 83.82 0) (unit 1)
+    (in_bom yes) (on_board yes) (dnp no) (fields_autoplaced)
+    (property "Reference" "#PWR09" (at 106.68 90.17 0)
+      (effects (font (size 1.27 1.27)) hide)
+    )
+    (property "Value" "GND" (at 106.68 88.2634 0)
+      (effects (font (size 1.27 1.27)))
+    )
+    (property "Footprint" "" (at 106.68 83.82 0)
+      (effects (font (size 1.27 1.27)) hide)
+    )
+    (property "Datasheet" "" (at 106.68 83.82 0)
+      (effects (font (size 1.27 1.27)) hide)
+    )
+    (pin "1")
+    (instances
+      (project "porta-jelly"
+        (path "/10477f3c-6568-4c00-b643-b8ffee73b374"
+          (reference "#PWR09") (unit 1)
+        )
+      )
+      (project "12v-jelly"
+        (path "/a6bbc090-914d-4858-aeca-5d2d4d192127"
+          (reference "#PWR03") (unit 1)
+        )
+      )
+      (project ""
+        (path "/d350497a-baf4-4270-a560-45c7bc5aa03e"
+          (reference "#PWR09") (unit 1)
+        )
+      )
