File: 12v-jelly.kicad_sch (KiCad schematic)
At the start: 32 parts, among them J1 PWR, J10 8, J3 1, J4 2, J5 3, J6 4, J7 5, J8 6, J9 7, Q1 DMP2022LSS-13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

Commit message: Part numbers
Parts:
- Q1: LCSC (none) -> C154919
- Q2: LCSC (none) -> C916396
- SW2: LCSC (none) -> C455107
Changed lines of the file:
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@@
+      (effects (font (size 1.27 1.27)) hide)
+    )
+    (property "LCSC" "C154919" (at 106.68 68.58 90)
       (effects (font (size 1.27 1.27)) hide)
     )
@@
     (property "Datasheet" "https://www.onsemi.com/pub/Collateral/NDS7002A-D.PDF" (at 109.22 78.74 0)
       (effects (font (size 1.27 1.27)) (justify left) hide)
+    )
+    (property "LCSC" "C916396" (at 109.22 78.74 0)
+      (effects (font (size 1.27 1.27)) hide)
     )
     (pin "1")
@@
       (effects (font (size 1.27 1.27)) hide)
     )
+    (property "LCSC" "C455107" (at 72.39 30.48 90)
+      (effects (font (size 1.27 1.27)) hide)
+    )
